File: hardware/pcb/PocketStockV2.kicad_pcb (KiCad board)
At the start: 4 copper layers, 31 x 40 mm, 7 parts, among them U1 C3_SuperMIni, U2 SSD1306

Commit message: Add full KiCad project and STEP model
Other:
- board text added: "designed by dior sausage"
- board text removed: "made by dior sausage"
Changed lines of the file:
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@@
 		(13 "F.Paste" user)
 		(15 "B.Paste" user)
-		(5 "F.SilkS" user)
-		(7 "B.SilkS" user)
+		(5 "F.SilkS" user "F.Silkscreen")
+		(7 "B.SilkS" user "B.Silkscreen")
 		(1 "F.Mask" user)
 		(3 "B.Mask" user)
 		(25 "Edge.Cuts" user)
 		(27 "Margin" user)
-		(31 "F.CrtYd" user)
-		(29 "B.CrtYd" user)
+		(31 "F.CrtYd" user "F.Courtyard")
+		(29 "B.CrtYd" user "B.Courtyard")
 		(35 "F.Fab" user)
 	)
@@
 			(plot_on_all_layers_selection 0x00000000_00000000_00000000_00000000)
 			(disableapertmacros no)
-			(usegerberextensions no)
-			(usegerberattributes yes)
-			(usegerberadvancedattributes yes)
-			(creategerberjobfile yes)
+			(usegerberextensions yes)
+			(usegerberattributes no)
+			(usegerberadvancedattributes no)
+			(creategerberjobfile no)
 			(dashed_line_dash_ratio 12.000000)
 			(dashed_line_gap_ratio 3.000000)
@@
 			(outputformat 1)
 			(mirror no)
-			(drillshape 1)
+			(drillshape 0)
 			(scaleselection 1)
-			(outputdirectory "")
+			(outputdirectory "gerbers/")
 		)
 	)
@@
 		)
 		(embedded_fonts no)
+		(model "/Users/armanaryafar/Downloads/0-96-inch-oled-lcd-module-4-pin-128x64-1/ssd1306 step.step"
+			(offset
+				(xyz 0 0 0)
+			)
+			(scale
+				(xyz 1 1 1)
+			)
+			(rotate
+				(xyz -90 -0 -0)
+			)
+		)
 	)
 	(footprint "LOGO"
@@
 		)
 		(embedded_fonts no)
+		(model "/Users/armanaryafar/Downloads/esp32-c3-supermini-1/ESP32-C3 supermini v5.step"
+			(offset
+				(xyz -20 -6 -3.5)
+			)
+			(scale
+				(xyz 1 1 1)
+			)
+			(rotate
+				(xyz 90 -180 -0)
+			)
+		)
 	)
 	(gr_line
@@
 		)
 	)
+	(gr_text "PocketStock V1"
+		(at 155.8 110.8 0)
+		(layer "F.SilkS")
+		(effects
+			(font
+				(size 1.524 1.524)
+				(thickness 0.3048)
+				(bold yes)
+			)
+			(justify left bottom)
+		)
+	)
 	(gr_text "SSD1306"
 		(at 159.6 94.4 0)
@@
 		)
 	)
-	(gr_text "made by dior sausage"
+	(gr_text "designed by dior sausage"
 		(at 173.8 110.3 0)
 		(layer "B.SilkS")
@@
 		)
 	)
-	(gr_text "PocketStock V1"
-		(at 155.8 110.8 0)
-		(layer "F.Paste")
-		(effects
-			(font
-				(size 1.524 1.524)
-				(thickness 0.3048)
-				(bold yes)
-			)
-			(justify left bottom)
-		)
-	)
